Commit message: Added working basic safety layer launch

File: src/lidar_launch/config/truck.urdf (robot description, URDF)
Before this commit: robot truck, 2 links, 1 joints
Links:
- link base_link: geometry visual mesh filename=package://lidar_launch/config/Truck_Model.stl scale=2.5 2.5 2.5

Commit message: Roi aangepast. sensor_offset_x toegevoegd. emergency_hold_sec en hazard_hold_sec aangepast. en visualisatie aangepast zodat het klopt met afstand. afstand is ook gecheckt. Deze werkt!

File: src/lidar_launch/config/truck.urdf (robot description, URDF)
Before this commit: robot truck, 2 links, 1 joints
Links:
- added link safety_base
- link base_link: geometry visual box size=5.0 0.75 1.3
- link velodyne: geometry visual cylinder length=0.072 radius=0.052
Joints:
- removed joint truck_to_lidar
- added joint base_link_to_safety_base: type fixed, parent base_link, child safety_base, origin xyz=0 0 0 rpy=0 0 0
- added joint safety_base_to_velodyne: type fixed, parent safety_base, child velodyne, origin xyz=-0.57 0.0 1.8 rpy=0 0 0
